File: GND-LIFT/GND-LIFT/GND-LIFT.kicad_sch (KiCad schematic)
At the start: 5 parts, among them J1 8191, J2 8191

Commit message: fix gnd-lift - add gerbers for gnd-lift & t-gnd
Connections:
- net CHASSIS: now also C1.2, J2.1 (Pin_1), R1.2; no longer C1.1, J1.1 (Pin_1), R1.1
- net PSU0V: now also C1.1, J1.1 (Pin_1), R1.1; no longer C1.2, J2.1 (Pin_1), R1.2
Other:
- moved on the sheet: C1, J1, J2, R1
Changed lines of the file:
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@@
 (kicad_sch (version 20230121) (generator eeschema)
   (paper "A4")
+  (junction (at 91.44 72.39) (diameter 0) (color 0 0 0 0)
+  )
+  (junction (at 91.44 92.71) (diameter 0) (color 0 0 0 0)
+  )
   (junction (at 154.94 82.55) (diameter 0) (color 0 0 0 0)
   )
   (junction (at 107.95 92.71) (diameter 0) (color 0 0 0 0)
   )
-  (junction (at 107.95 111.76) (diameter 0) (color 0 0 0 0)
-  )
-  (junction (at 91.44 92.71) (diameter 0) (color 0 0 0 0)
-  )
   (junction (at 123.19 111.76) (diameter 0) (color 0 0 0 0)
   )
-  (junction (at 91.44 72.39) (diameter 0) (color 0 0 0 0)
+  (junction (at 107.95 111.76) (diameter 0) (color 0 0 0 0)
   )
   (wire (pts (xy 91.44 111.76) (xy 107.95 111.76))
     (stroke (width 0) (type default))
   )
-  (wire (pts (xy 123.19 82.55) (xy 123.19 111.76))
+  (wire (pts (xy 154.94 82.55) (xy 156.21 82.55))
     (stroke (width 0) (type default))
   )
-  (wire (pts (xy 107.95 92.71) (xy 107.95 96.52))
+  (wire (pts (xy 123.19 82.55) (xy 123.19 111.76))
     (stroke (width 0) (type default))
   )
@@
     (stroke (width 0) (type default))
   )
-  (wire (pts (xy 91.44 104.14) (xy 91.44 111.76))
-    (stroke (width 0) (type default))
-  )
   (wire (pts (xy 127 82.55) (xy 123.19 82.55))
     (stroke (width 0) (type default))
@@
     (stroke (width 0) (type default))
   )
-  (wire (pts (xy 91.44 92.71) (xy 91.44 96.52))
+  (wire (pts (xy 88.9 72.39) (xy 91.44 72.39))
+    (stroke (width 0) (type default))
+  )
+  (wire (pts (xy 107.95 111.76) (xy 123.19 111.76))
+    (stroke (width 0) (type default))
+  )
+  (wire (pts (xy 91.44 105.41) (xy 91.44 111.76))
     (stroke (width 0) (type default))
   )
@@
     (stroke (width 0) (type default))
   )
-  (wire (pts (xy 107.95 111.76) (xy 123.19 111.76))
-    (stroke (width 0) (type default))
-  )
-  (wire (pts (xy 107.95 104.14) (xy 107.95 111.76))
-    (stroke (width 0) (type default))
-  )
-  (wire (pts (xy 154.94 82.55) (xy 158.75 82.55))
-    (stroke (width 0) (type default))
-  )
-  (wire (pts (xy 91.44 72.39) (xy 90.17 72.39))
-    (stroke (width 0) (type default))
-  )
-  (wire (pts (xy 107.95 92.71) (xy 91.44 92.71))
-    (stroke (width 0) (type default))
-  )
-  (wire (pts (xy 134.62 92.71) (xy 107.95 92.71))
+  (wire (pts (xy 91.44 92.71) (xy 107.95 92.71))
     (stroke (width 0) (type default))
   )
   (wire (pts (xy 142.24 82.55) (xy 154.94 82.55))
+    (stroke (width 0) (type default))
+  )
+  (wire (pts (xy 107.95 92.71) (xy 134.62 92.71))
+    (stroke (width 0) (type default))
+  )
+  (wire (pts (xy 107.95 106.68) (xy 107.95 111.76))
+    (stroke (width 0) (type default))
+  )
+  (wire (pts (xy 107.95 92.71) (xy 107.95 99.06))
+    (stroke (width 0) (type default))
+  )
+  (wire (pts (xy 91.44 92.71) (xy 91.44 97.79))
     (stroke (width 0) (type default))
   )
@@
     )
   )
-  (symbol (lib_id "Device:R") (at 91.44 100.33 0) (unit 1)
+  (symbol (lib_id "Device:R") (at 91.44 101.6 180) (unit 1)
     (in_bom yes) (on_board yes) (dnp no) (fields_autoplaced)
-    (property "Reference" "R1" (at 93.98 99.06 0)
-      (effects (font (size 1.27 1.27)) (justify left))
+    (property "Reference" "R1" (at 93.98 100.33 0)
+      (effects (font (size 1.27 1.27)) (justify right))
     )
-    (property "Value" "10R 5W" (at 93.98 101.6 0)
-      (effects (font (size 1.27 1.27)) (justify left))
+    (property "Value" "10R 5W" (at 93.98 102.87 0)
+      (effects (font (size 1.27 1.27)) (justify right))
     )
-    (property "Footprint" "CustomKicadFootprint:VishayAC05" (at 89.662 100.33 90)
+    (property "Footprint" "CustomKicadFootprint:VishayAC05" (at 93.218 101.6 90)
       (effects (font (size 1.27 1.27)) hide)
     )
-    (property "Datasheet" "~" (at 91.44 100.33 0)
+    (property "Datasheet" "~" (at 91.44 101.6 0)
       (effects (font (size 1.27 1.27)) hide)
     )
@@
     )
   )
-  (symbol (lib_id "Connector:Screw_Terminal_01x01") (at 163.83 82.55 0) (unit 1)
+  (symbol (lib_id "Connector:Screw_Terminal_01x01") (at 83.82 72.39 180) (unit 1)
     (in_bom yes) (on_board yes) (dnp no) (fields_autoplaced)
-    (property "Reference" "J2" (at 166.37 81.28 0)
-      (effects (font (size 1.27 1.27)) (justify left))
+    (property "Reference" "J2" (at 83.82 66.04 0)
+      (effects (font (size 1.27 1.27)))
     )
-    (property "Value" "8191" (at 166.37 83.82 0)
-      (effects (font (size 1.27 1.27)) (justify left))
+    (property "Value" "8191" (at 83.82 68.58 0)
+      (effects (font (size 1.27 1.27)))
     )
-    (property "Footprint" "CustomKicadFootprint:KEYSTONE_8191" (at 163.83 82.55 0)
+    (property "Footprint" "CustomKicadFootprint:KEYSTONE_8191" (at 83.82 72.39 0)
       (effects (font (size 1.27 1.27)) hide)
     )
-    (property "Datasheet" "~" (at 163.83 82.55 0)
+    (property "Datasheet" "~" (at 83.82 72.39 0)
       (effects (font (size 1.27 1.27)) hide)
     )
@@
     )
   )
-  (symbol (lib_id "Device:C") (at 107.95 100.33 0) (unit 1)
+  (symbol (lib_id "Device:C") (at 107.95 102.87 180) (unit 1)
     (in_bom yes) (on_board yes) (dnp no) (fields_autoplaced)
-    (property "Reference" "C1" (at 111.76 99.06 0)
-      (effects (font (size 1.27 1.27)) (justify left))
+    (property "Reference" "C1" (at 111.76 101.6 0)
+      (effects (font (size 1.27 1.27)) (justify right))
     )
-    (property "Value" "100n" (at 111.76 101.6 0)
-      (effects (font (size 1.27 1.27)) (justify left))
+    (property "Value" "100n" (at 111.76 104.14 0)
+      (effects (font (size 1.27 1.27)) (justify right))
     )
-    (property "Footprint" "Capacitor_THT:C_Rect_L13.0mm_W6.0mm_P10.00mm_FKS3_FKP3_MKS4" (at 108.9152 104.14 0)
+    (property "Footprint" "Capacitor_THT:C_Rect_L13.0mm_W6.0mm_P10.00mm_FKS3_FKP3_MKS4" (at 106.9848 99.06 0)
       (effects (font (size 1.27 1.27)) hide)
     )
-    (property "Datasheet" "~" (at 107.95 100.33 0)
+    (property "Datasheet" "~" (at 107.95 102.87 0)
       (effects (font (size 1.27 1.27)) hide)
     )
@@
     )
   )
-  (symbol (lib_id "Connector:Screw_Terminal_01x01") (at 85.09 72.39 180) (unit 1)
+  (symbol (lib_id "Connector:Screw_Terminal_01x01") (at 161.29 82.55 0) (unit 1)
     (in_bom yes) (on_board yes) (dnp no) (fields_autoplaced)
-    (property "Reference" "J1" (at 85.09 66.04 0)
-      (effects (font (size 1.27 1.27)))
+    (property "Reference" "J1" (at 163.83 81.28 0)
+      (effects (font (size 1.27 1.27)) (justify left))
     )
-    (property "Value" "8191" (at 85.09 68.58 0)
-      (effects (font (size 1.27 1.27)))
+    (property "Value" "8191" (at 163.83 83.82 0)
+      (effects (font (size 1.27 1.27)) (justify left))
     )
-    (property "Footprint" "CustomKicadFootprint:KEYSTONE_8191" (at 85.09 72.39 0)
+    (property "Footprint" "CustomKicadFootprint:KEYSTONE_8191" (at 161.29 82.55 0)
       (effects (font (size 1.27 1.27)) hide)
     )
-    (property "Datasheet" "~" (at 85.09 72.39 0)
+    (property "Datasheet" "~" (at 161.29 82.55 0)
       (effects (font (size 1.27 1.27)) hide)
     )
