File: torpedo-iii/torpedo-iii/torpedo-iii-left.kicad_sch (KiCad schematic)
At the start: 46 parts, among them J1 NMJ6HCD2, J2 5.08mm Terminal, J3 5.08mm Terminal, J4 5.08mm Terminal, J5 5.08mm Terminal, Q101 KSP42, Q102 2SC4793, Q103 DN2540N3-G, Q104 2SC4793, Q105 KSP42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

Commit message: update torpedo-iii
Parts:
- R109: value 268R -> 67R
- R110: value 2680R -> 670R
