File: torpedo-iii/torpedo-iii/torpedo-iii-right.kicad_sch (KiCad schematic)
At the start: 38 parts, among them Q201 KSP42, Q202 2SC4793, Q203 DN2540N3-G, Q204 2SC4793, Q205 KSP42, T201 Cinemag, U201 12AY7, U202 LM334Z, U203 LM334Z, U204 LM334Z

Commit message: update torpedo-iii
Parts:
- R209: value 26.8R -> 67R
- R210: value 2680R -> 670R
