File: wolverine-protection/wolverine_protection/wolverine_protection.kicad_pcb (KiCad board)
At the start: 2 copper layers, 30 parts, among them J1 8191, J2 8191, J3 8191, J4 8191, Q1 027N10N, Q2 027N10N, Q3 MMBT3904, U1 STM32G030K6Tx, U2 LM317_TO-220, U3 VOM1271T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

Commit message: update wolverine 16-07-24
Parts:
- added C8: 2.2u, Capacitor_SMD:C_1206_3216Metric, F.Cu at (185.4, 64.6)
- added D4: 1N4148W, Diode_SMD:D_SOD-123, F.Cu at (195.6, 81.3)
- added D5: 1N4148W, Diode_SMD:D_SOD-123, F.Cu at (198.1, 81.4)
- added D6: LED, LED_SMD:LED_0805_2012Metric, F.Cu at (88.9, 80.1)
- added D7: LED, LED_SMD:LED_0805_2012Metric, F.Cu at (91.4, 80.1)
- added D8: LED, LED_SMD:LED_0805_2012Metric, F.Cu at (86.4, 80.1)
- added D9: LED, LED_SMD:LED_0805_2012Metric, F.Cu at (83.8, 80.1)
- added J5: JST XH, Connector_JST:JST_XH_B2B-XH-A_1x02_P2.50mm_Vertical, F.Cu at (238.2, 60.0)
- added J6: 8191, CustomKicadFootprint:KEYSTONE_8191, F.Cu at (190.5, 45.8)
- added J7: JST XH, Connector_JST:JST_XH_B2B-XH-A_1x02_P2.50mm_Vertical, F.Cu at (238.2, 67.8)
- added J8: JST XH, Connector_JST:JST_XH_B2B-XH-A_1x02_P2.50mm_Vertical, F.Cu at (238.2, 75.5)
- added J9: JST XH, Connector_JST:JST_XH_B2B-XH-A_1x02_P2.50mm_Vertical, F.Cu at (238.2, 83.3)
- added Q4: BC549, Package_TO_SOT_THT:TO-92_Inline_Wide, F.Cu at (195.6, 76.2)
- added Q5: 2N5551, Package_TO_SOT_THT:TO-92_Inline_Wide, F.Cu at (200.7, 76.2)
- added R10: 470R, Resistor_SMD:R_1206_3216Metric, F.Cu at (180.3, 64.6)
- added R11: 18k, Resistor_SMD:R_1206_3216Metric, F.Cu at (193.0, 81.3)
- added R12: 18k, Resistor_SMD:R_1206_3216Metric, F.Cu at (200.7, 81.3)
- added R13: 220R, Resistor_SMD:R_1206_3216Metric, F.Cu at (203.2, 81.3)
- added R14: 4.7k, Resistor_SMD:R_1206_3216Metric, F.Cu at (218.4, 71.1)
- added R15: 4.7k, Resistor_SMD:R_1206_3216Metric, F.Cu at (248.7, 54.9)
- added R16: 4.7k, Resistor_SMD:R_1206_3216Metric, F.Cu at (254.3, 41.8)
- added R17: 140R, Resistor_SMD:R_1206_3216Metric, F.Cu at (88.9, 75.1)
- added R18: 140R, Resistor_SMD:R_1206_3216Metric, F.Cu at (91.4, 75.1)
- added R19: 140R, Resistor_SMD:R_1206_3216Metric, F.Cu at (86.4, 75.1)
- added R20: 108R, Resistor_SMD:R_1206_3216Metric, F.Cu at (83.8, 75.1)
- added R9: 470R, Resistor_SMD:R_1206_3216Metric, F.Cu at (182.9, 64.6)
- added U5: CNY17-3, Package_DIP:DIP-6_W7.62mm, F.Cu at (207.0, 68.6)
- C7: footprint Capacitor_SMD:C_1206_3216Metric -> Capacitor_THT:C_Radial_D12.5mm_H20.0mm_P5.00mm
- moved R1 167.0 mm to (237.5, 41.8)
- moved C3 119.9 mm to (129.5, 139.7)
- moved C6 115.9 mm to (142.2, 132.1)
- moved J3 111.8 mm to (50.8, 50.8)
- moved U6 110.8 mm to (64.8, 72.4), turned to -90 degrees
- moved C7 109.9 mm to (63.5, 66.0), turned to 90 degrees
- moved D2 103.1 mm to (129.5, 134.6), turned to -90 degrees
- moved D1 101.1 mm to (129.5, 127.0), turned to -90 degrees
- moved R8 93.7 mm to (71.1, 71.1), turned to 90 degrees
- moved R6 92.4 mm to (114.3, 76.2)
- moved J2 90.4 mm to (50.8, 76.2)
- moved Q3 89.0 mm to (115.9, 81.3), turned to 0 degrees
- moved R7 87.8 mm to (68.6, 71.1), turned to -90 degrees
- moved C1 83.1 mm to (99.1, 121.9), turned to -90 degrees
- moved U2 82.5 mm to (134.6, 128.6)
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