File: wolverine-protection/wolverine_protection/wolverine_protection.kicad_sch (KiCad schematic)
At the start: 57 parts, among them J1 8191, J2 8191, J3 8191, J4 8191, J5 JST XH, J6 8191, J7 JST XH, J8 JST XH, J9 JST XH, Q1 027N10N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

Commit message: update wolverine 16-07-24
Parts:
- C7: footprint Capacitor_SMD:C_1206_3216Metric -> Capacitor_THT:C_Radial_D12.5mm_H20.0mm_P5.00mm
- C8: footprint Capacitor_THT:CP_Radial_D13.0mm_P5.00mm -> Capacitor_SMD:C_1206_3216Metric
- U5: footprint (none) -> Package_DIP:DIP-6_W7.62mm
Changed lines of the file:
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@@
 			)
 		)
-		(property "Footprint" "Capacitor_SMD:C_1206_3216Metric"
+		(property "Footprint" "Capacitor_THT:C_Radial_D12.5mm_H20.0mm_P5.00mm"
 			(at 210.5152 58.42 0)
 			(effects
@@
 			)
 		)
-		(property "Footprint" ""
+		(property "Footprint" "Package_DIP:DIP-6_W7.62mm"
 			(at 151.13 158.75 0)
 			(effects
@@
 			)
 		)
-		(property "Footprint" "Capacitor_THT:CP_Radial_D13.0mm_P5.00mm"
+		(property "Footprint" "Capacitor_SMD:C_1206_3216Metric"
 			(at 92.4052 220.98 0)
 			(effects
